Commit message: fix(capsule): one circle per cross-section plane -> few mergeable capsules
A plane cuts multiple contour loops on flanged links -> multiple circles ->
messy pairing -> 97 unmergeable short capsules. Group contours by plane, fit ONE
circle (MEC of all loop points) per plane -> uniform across planes -> consecutive
capsules share endpoints -> mergeCollinear collapses each link to ~1 long
capsule. FR3: 13 capsules (1/link, fingers 2), all covered.

File: resources/fr3/urdf/fr3_capsuleized.urdf (robot description, URDF)
Before this commit: robot bot, 14 links, 13 joints
Links:
- link fr3_link0: geometry collision cylinder length=0.239863 radius=0.107104; collision sphere radius=0.107104
- link fr3_link1: geometry collision cylinder length=0.284383 radius=0.080738; collision sphere radius=0.080738
- link fr3_link2: geometry collision cylinder length=0.285592 radius=0.080391; collision sphere radius=0.080391
- link fr3_link3: geometry collision cylinder length=0.254614 radius=0.075502; collision sphere radius=0.075502
- link fr3_link4: geometry collision cylinder length=0.256383 radius=0.076085; collision sphere radius=0.076085
- link fr3_link5: geometry collision cylinder length=0.343367 radius=0.073151; collision sphere radius=0.073151
- link fr3_link6: geometry collision cylinder length=0.185416 radius=0.075958; collision sphere radius=0.075958
- link fr3_link7: geometry collision cylinder length=0.142033 radius=0.050662; collision sphere radius=0.050662
- link hand_hand: geometry collision cylinder length=0.206419 radius=0.048119; collision sphere radius=0.048119
- link hand_leftfinger: geometry collision cylinder length=0.048333 radius=0.013789; collision cylinder length=0.080494 radius=0.026123
- link hand_rightfinger: geometry collision cylinder length=0.048333 radius=0.013789; collision cylinder length=0.080494 radius=0.026123
