Commit message: assets: regenerate FR3 tight capsule output

File: resources/fr3/urdf/fr3_capsuleized.urdf (robot description, URDF)
Before this commit: robot bot, 14 links, 13 joints
Links:
- link fr3_link0: geometry collision cylinder length=0.035936 radius=0.072194; collision cylinder length=0.203636 radius=0.107683
- link fr3_link1: geometry collision cylinder length=0.071458 radius=0.064088; collision cylinder length=0.212749 radius=0.085190
- link fr3_link2: geometry collision cylinder length=0.285214 radius=0.085889; collision sphere radius=0.085889
- link fr3_link3: geometry collision cylinder length=0.254222 radius=0.079442; collision sphere radius=0.079442
- link fr3_link4: geometry collision cylinder length=0.255957 radius=0.079450; collision sphere radius=0.079450
- link fr3_link5: geometry collision cylinder length=0.343345 radius=0.072580; collision sphere radius=0.072580
- link fr3_link6: geometry collision cylinder length=0.185485 radius=0.076478; collision sphere radius=0.076478
- link fr3_link7: geometry collision cylinder length=0.035579 radius=0.038466; collision cylinder length=0.106473 radius=0.050865
- link hand_hand: geometry collision cylinder length=0.206423 radius=0.049001; collision sphere radius=0.049001
- link hand_leftfinger: geometry collision cylinder length=0.021511 radius=0.014643; collision cylinder length=0.032222 radius=0.011853
- link hand_rightfinger: geometry collision cylinder length=0.021511 radius=0.014643; collision cylinder length=0.032222 radius=0.011853

Commit message: docs: document capsule endpoint center semantics

File: resources/fr3/urdf/fr3_capsuleized.urdf (robot description, URDF)
Before this commit: robot bot, 14 links, 13 joints
Links:
- link fr3_link0: geometry collision cylinder length=0.073671 radius=0.107683; collision sphere radius=0.107683
- link fr3_link1: geometry collision cylinder length=0.004647 radius=0.071244; collision cylinder length=0.133841 radius=0.085299
- link fr3_link2: geometry collision cylinder length=0.148798 radius=0.086811; collision sphere radius=0.086811
- link fr3_link3: geometry collision cylinder length=0.115592 radius=0.079753; collision sphere radius=0.079753
- link fr3_link4: geometry collision cylinder length=0.116163 radius=0.079916; collision sphere radius=0.079916
- link fr3_link5: geometry collision cylinder length=0.227397 radius=0.072580; collision sphere radius=0.072580
- link fr3_link6: geometry collision cylinder length=0.071069 radius=0.076478; collision sphere radius=0.076478
- link fr3_link7: geometry collision cylinder length=0.002390 radius=0.042971; collision cylinder length=0.042026 radius=0.050873
- link hand_hand: geometry collision cylinder length=0.141655 radius=0.049001; collision sphere radius=0.049001
- link hand_leftfinger: geometry collision cylinder length=0.012071 radius=0.027077; collision cylinder length=0.016366 radius=0.026186
- link hand_rightfinger: geometry collision cylinder length=0.012071 radius=0.027077; collision cylinder length=0.016366 radius=0.026186
