Commit message: chore: regenerate fr3_compare_bundle with union-volume capsules
Regenerated via compare-all --mesh-source visual. Capsule URDFs
now reflect union-volume fitting; all meshes reference converted
.obj files from the .dae visual mesh pre-pass.

File: assets/fr3_compare_bundle/fr3_capsule_default.urdf (robot description, URDF)
Before this commit: robot bot, 14 links, 13 joints
Links:
- link fr3_link5: geometry collision cylinder length=0.024224 radius=0.052032; collision cylinder length=0.039832 radius=0.068770
- link fr3_link6: geometry collision cylinder length=0.000078 radius=0.089993; collision cylinder length=0.065965 radius=0.090288
- link hand_leftfinger: geometry collision cylinder length=0.007463 radius=0.025740; collision cylinder length=0.014368 radius=0.026280
- link hand_rightfinger: geometry collision cylinder length=0.007463 radius=0.025740; collision cylinder length=0.014368 radius=0.026280

File: assets/fr3_compare_bundle/fr3_capsule_high_detail.urdf (robot description, URDF)
Before this commit: robot bot, 14 links, 13 joints
Links:
- link fr3_link5: geometry collision cylinder length=0.001778 radius=0.056454; collision cylinder length=0.007678 radius=0.047721
- link fr3_link6: geometry collision cylinder length=0.006775 radius=0.067779; collision cylinder length=0.049296 radius=0.089170
- link fr3_link7: geometry collision cylinder length=0.000873 radius=0.040932; collision cylinder length=0.042725 radius=0.051855

File: assets/fr3_compare_bundle/fr3_convex.urdf (robot description, URDF)
Before this commit: robot bot, 14 links, 13 joints
Links:
- link fr3_link0: geometry collision mesh filename=meshes/link0_1.obj; visual mesh filename=meshes/link0.dae
- link fr3_link1: geometry collision mesh filename=meshes/link1_1.obj; visual mesh filename=meshes/link1.dae
- link fr3_link2: geometry collision mesh filename=meshes/link2_1.obj; visual mesh filename=meshes/link2.dae
- link fr3_link3: geometry collision mesh filename=meshes/link3_1.obj; visual mesh filename=meshes/link3.dae
- link fr3_link4: geometry collision mesh filename=meshes/link4_1.obj; visual mesh filename=meshes/link4.dae
- link fr3_link5: geometry collision mesh filename=meshes/link5_1.obj; visual mesh filename=meshes/link5.dae
- link fr3_link6: geometry collision mesh filename=meshes/link6_1.obj; visual mesh filename=meshes/link6.dae
- link fr3_link7: geometry collision mesh filename=meshes/link7_1.obj; visual mesh filename=meshes/link7.dae
- link hand_hand: geometry collision mesh filename=meshes/hand_1.obj; visual mesh filename=meshes/hand.dae
- link hand_leftfinger: geometry collision mesh filename=meshes/flex_griper_connect_1.obj; visual mesh filename=meshes/flex_griper_connect.stl
- link hand_rightfinger: geometry collision mesh filename=meshes/flex_griper_connect_1.obj; visual mesh filename=meshes/flex_griper_connect.stl

File: assets/fr3_compare_bundle/fr3_sphere_default.urdf (robot description, URDF)
Before this commit: robot bot, 14 links, 13 joints
Links:
- link fr3_link0: geometry collision sphere radius=0.022296; collision sphere radius=0.024740
- link fr3_link1: geometry collision sphere radius=0.012660; collision sphere radius=0.041934
- link fr3_link2: geometry collision sphere radius=0.026841; collision sphere radius=0.039931
- link fr3_link3: geometry collision sphere radius=0.018411; collision sphere radius=0.027189
- link fr3_link4: geometry collision sphere radius=0.014219; collision sphere radius=0.032887
- link fr3_link5: geometry collision sphere radius=0.038453; collision sphere radius=0.038470
- link fr3_link6: geometry collision sphere radius=0.028540; collision sphere radius=0.039288
- link fr3_link7: geometry collision sphere radius=0.019152; collision sphere radius=0.023712
- link hand_hand: geometry collision sphere radius=0.033738; collision sphere radius=0.035113
- link hand_leftfinger: geometry collision sphere radius=0.013449; collision sphere radius=0.015415
- link hand_rightfinger: geometry collision sphere radius=0.011975; collision sphere radius=0.015011

File: assets/fr3_compare_bundle/fr3_sphere_single.urdf (robot description, URDF)
Before this commit: robot bot, 14 links, 13 joints
Links:
- link fr3_link0: geometry collision sphere radius=0.128383; visual mesh filename=meshes/link0.dae
- link fr3_link1: geometry collision sphere radius=0.144564; visual mesh filename=meshes/link1.dae
- link fr3_link2: geometry collision sphere radius=0.144056; visual mesh filename=meshes/link2.dae
- link fr3_link3: geometry collision sphere radius=0.127649; visual mesh filename=meshes/link3.dae
- link fr3_link4: geometry collision sphere radius=0.127667; visual mesh filename=meshes/link4.dae
- link fr3_link5: geometry collision sphere radius=0.173477; visual mesh filename=meshes/link5.dae
- link fr3_link6: geometry collision sphere radius=0.098992; visual mesh filename=meshes/link6.dae
- link fr3_link7: geometry collision sphere radius=0.072815; visual mesh filename=meshes/link7.dae
- link hand_hand: geometry collision sphere radius=0.107798; visual mesh filename=meshes/hand.dae
- link hand_rightfinger: geometry collision sphere radius=0.064548; visual mesh filename=meshes/flex_griper_connect.stl
